File: files/_autosave-address.kicad_sch (KiCad schematic)
At the start: 4 parts, among them J1 VLB_slot, U1 86C375

Commit message: PCB work
Parts:
- U1: value 86C375 -> 86C325
Changed lines of the file:
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@@
       (effects (font (size 1.524 1.524)))
     )
-    (property "Value" "86C375" (at 137.16 86.36 0)
+    (property "Value" "86C325" (at 137.16 86.36 0)
       (effects (font (size 1.524 1.524)))
     )
@@
       (effects (font (size 1.524 1.524)) (justify left))
     )
-    (property "Value" "86C375" (at 220.98 135.255 0)
+    (property "Value" "86C325" (at 220.98 135.255 0)
       (effects (font (size 1.524 1.524)) (justify left))
     )
@@
       (effects (font (size 1.524 1.524)))
     )
-    (property "Value" "86C375" (at 136.525 143.51 0)
+    (property "Value" "86C325" (at 136.525 143.51 0)
       (effects (font (size 1.524 1.524)))
     )
