File: files/virge-vlb.kicad_pcb (KiCad board)
At the start: 2 copper layers, 240.5 x 121.5 mm, 15 parts, among them J1 VLB_slot, U1 86C375_layout, U2 27C010, U5 74F08, U6 74F08

Commit message: changed memory chips, more progress
Parts:
- added C1: 10pF, Capacitor_SMD:C_0805_2012Metric_Pad1.18x1.45mm_HandSolder, F.Cu at (76.0, 105.0)
- added C2: 10pF, Capacitor_SMD:C_0805_2012Metric_Pad1.18x1.45mm_HandSolder, F.Cu at (76.0, 108.0)
- added C3: 10pF, Capacitor_SMD:C_0805_2012Metric_Pad1.18x1.45mm_HandSolder, F.Cu at (259.2, 64.1)
- added C4: 10pF, Capacitor_SMD:C_0805_2012Metric_Pad1.18x1.45mm_HandSolder, F.Cu at (259.1, 72.5)
- added C5: 10pF, Capacitor_SMD:C_0805_2012Metric_Pad1.18x1.45mm_HandSolder, F.Cu at (259.1, 75.5)
- added C6: 10pF, Capacitor_SMD:C_0805_2012Metric_Pad1.18x1.45mm_HandSolder, F.Cu at (259.1, 78.5)
- added C7: 10pF, Capacitor_SMD:C_0805_2012Metric_Pad1.18x1.45mm_HandSolder, F.Cu at (259.1, 81.5)
- added C8: 10pF, Capacitor_SMD:C_0805_2012Metric_Pad1.18x1.45mm_HandSolder, F.Cu at (259.1, 84.5)
- added C9: 0.1uF, Capacitor_SMD:C_0805_2012Metric_Pad1.18x1.45mm_HandSolder, F.Cu at (259.1, 87.5)
- added J2: VGA, Connector_Dsub:DSUB-15-HD_Female_Horizontal_P2.29x1.98mm_EdgePinOffset8.35mm_Housed_MountingHolesOffset10.89mm, F.Cu at (270.3, 75.9)
- added J3: VESA feature, Connector_PinHeader_2.54mm:PinHeader_2x13_P2.54mm_Vertical, F.Cu at (56.1, 59.0)
- added JP1: Conn_01x02, Connector_PinHeader_2.54mm:PinHeader_1x02_P2.54mm_Vertical, F.Cu at (215.1, 38.0)
- added JP2: IRQ select, Connector_PinHeader_2.54mm:PinHeader_1x03_P2.54mm_Vertical, F.Cu at (207.8, 26.3)
- added R1: 75R, Resistor_SMD:R_0805_2012Metric_Pad1.20x1.40mm_HandSolder, F.Cu at (76.0, 82.1)
- added R10: 33R, Resistor_SMD:R_0805_2012Metric_Pad1.20x1.40mm_HandSolder, F.Cu at (144.8, 112.5)
- added R11: 10K, Resistor_SMD:R_0805_2012Metric, F.Cu at (118.3, 72.5)
- added R11: 33R, Resistor_SMD:R_0805_2012Metric_Pad1.20x1.40mm_HandSolder, F.Cu at (144.8, 115.4)
- added R12: 33R, Resistor_SMD:R_0805_2012Metric_Pad1.20x1.40mm_HandSolder, F.Cu at (149.6, 100.7)
- added R13: 33R, Resistor_SMD:R_0805_2012Metric_Pad1.20x1.40mm_HandSolder, F.Cu at (149.6, 103.6)
- added R14: 33R, Resistor_SMD:R_0805_2012Metric_Pad1.20x1.40mm_HandSolder, F.Cu at (149.6, 106.5)
- added R15: 33R, Resistor_SMD:R_0805_2012Metric_Pad1.20x1.40mm_HandSolder, F.Cu at (149.6, 109.5)
- added R16: 33R, Resistor_SMD:R_0805_2012Metric_Pad1.20x1.40mm_HandSolder, F.Cu at (149.6, 112.5)
- added R17: 100R, Resistor_SMD:R_0805_2012Metric_Pad1.20x1.40mm_HandSolder, F.Cu at (144.8, 120.3)
- added R18: 33R, Resistor_SMD:R_0805_2012Metric_Pad1.20x1.40mm_HandSolder, F.Cu at (76.0, 96.8)
- added R19: 33R, Resistor_SMD:R_0805_2012Metric_Pad1.20x1.40mm_HandSolder, F.Cu at (76.0, 99.8)
- added R2: 75R, Resistor_SMD:R_0805_2012Metric_Pad1.20x1.40mm_HandSolder, F.Cu at (76.0, 85.0)
- added R20: 33R, Resistor_SMD:R_0805_2012Metric_Pad1.20x1.40mm_HandSolder, F.Cu at (80.7, 82.1)
- added R21: 33R, Resistor_SMD:R_0805_2012Metric_Pad1.20x1.40mm_HandSolder, F.Cu at (80.7, 85.0)
- added R22: 33R, Resistor_SMD:R_0805_2012Metric_Pad1.20x1.40mm_HandSolder, F.Cu at (80.7, 88.0)
- added R23: 33R, Resistor_SMD:R_0805_2012Metric_Pad1.20x1.40mm_HandSolder, F.Cu at (90.9, 104.6)
- added R24: 33R, Resistor_SMD:R_0805_2012Metric_Pad1.20x1.40mm_HandSolder, F.Cu at (80.7, 93.9)
- added R25: 33R, Resistor_SMD:R_0805_2012Metric_Pad1.20x1.40mm_HandSolder, F.Cu at (80.7, 96.8)
- added R26: 33R, Resistor_SMD:R_0805_2012Metric_Pad1.20x1.40mm_HandSolder, F.Cu at (80.7, 99.8)
- added R27: 4K7, Resistor_SMD:R_0805_2012Metric_Pad1.20x1.40mm_HandSolder, F.Cu at (85.5, 82.1)
- added R28: 33R, Resistor_SMD:R_0805_2012Metric_Pad1.20x1.40mm_HandSolder, F.Cu at (85.5, 85.0)
- added R29: 4K7, Resistor_SMD:R_0805_2012Metric_Pad1.20x1.40mm_HandSolder, F.Cu at (85.5, 88.0)
- added R3: 75R, Resistor_SMD:R_0805_2012Metric_Pad1.20x1.40mm_HandSolder, F.Cu at (76.0, 88.0)
- added R30: 33R, Resistor_SMD:R_0805_2012Metric_Pad1.20x1.40mm_HandSolder, F.Cu at (91.8, 96.0)
- added R31: 4K7, Resistor_SMD:R_0805_2012Metric_Pad1.20x1.40mm_HandSolder, F.Cu at (85.5, 93.9)
- added R32: 33R, Resistor_SMD:R_0805_2012Metric_Pad1.20x1.40mm_HandSolder, F.Cu at (85.5, 96.8)
- added R33: 150R, Resistor_SMD:R_0805_2012Metric_Pad1.20x1.40mm_HandSolder, F.Cu at (85.5, 99.8)
- added R4: 33R, Resistor_SMD:R_0805_2012Metric_Pad1.20x1.40mm_HandSolder, F.Cu at (243.8, 83.8)
- added R5: 33R, Resistor_SMD:R_0805_2012Metric_Pad1.20x1.40mm_HandSolder, F.Cu at (76.0, 93.9)
- added R6: 33R, Resistor_SMD:R_0805_2012Metric_Pad1.20x1.40mm_HandSolder, F.Cu at (144.8, 100.7)
- added R7: 33R, Resistor_SMD:R_0805_2012Metric_Pad1.20x1.40mm_HandSolder, F.Cu at (144.8, 103.6)
- added R8: 33R, Resistor_SMD:R_0805_2012Metric_Pad1.20x1.40mm_HandSolder, F.Cu at (144.8, 106.5)
- added R9: 33R, Resistor_SMD:R_0805_2012Metric_Pad1.20x1.40mm_HandSolder, F.Cu at (144.8, 109.5)
- added U10: 74F245, Package_SO:SO-20_5.3x12.6mm_P1.27mm, F.Cu at (249.4, 125.2)
- added U3: ~, VLB:SOJ-40_10.16x26.00mm_P1.27mm, F.Cu at (141.4, 66.2)
- added U4: ~, VLB:SOJ-40_10.16x26.00mm_P1.27mm, F.Cu at (154.1, 66.2)
- added Y1: 14.318MHz, Crystal:Crystal_HC18-U_Vertical, F.Cu at (96.7, 82.7)
- U1: value 86C375_layout -> 86C375
- U2: footprint Package_DIP:DIP-28_W15.24mm -> Package_DIP:DIP-32_W15.24mm
- U5, U6: value 74F08 -> ~; footprint Package_SO:SOIC-14_3.9x8.7mm_P1.27mm -> VLB:SOJ-40_10.16x26.00mm_P1.27mm
- moved U6 78.4 mm to (179.4, 66.2)
- moved U5 76.5 mm to (166.8, 66.2)
- moved R10 34.9 mm to (128.1, 84.8)
- moved R6 34.9 mm to (128.1, 73.0)
- moved R7 34.9 mm to (128.1, 76.0)
- moved R8 34.9 mm to (128.1, 79.0)
- moved R9 34.9 mm to (128.1, 81.9)
- moved R1 34.9 mm to (123.7, 73.0)
- moved R2 34.9 mm to (123.7, 76.0)
- moved R3 34.9 mm to (123.7, 79.0)
- moved R4 34.9 mm to (123.7, 81.9)
- moved R5 34.9 mm to (123.7, 84.8)
- moved U1 21.4 mm to (107.2, 109.9), turned to 90 degrees
- moved U2 12.0 mm to (254.5, 99.9)
- moved J1 1.68 mm to (121.9, 140.5)
Connections:
- net /ISA Bus/A0 renamed /ISA Bus/R_A0
- net /ISA Bus/A1 renamed /ISA Bus/R_A1
- net /ISA Bus/A10 renamed /ISA Bus/R_A10
- net /ISA Bus/A11 renamed /ISA Bus/R_A11
- net /ISA Bus/A12 renamed /ISA Bus/R_A12
- net /ISA Bus/A13 renamed /ISA Bus/R_A13
- net /ISA Bus/A15 renamed /ISA Bus/R_A15
- net /ISA Bus/A16 renamed /ISA Bus/R_A16
- net /ISA Bus/A2 renamed /ISA Bus/R_A2
- net /ISA Bus/A3 renamed /ISA Bus/R_A3
- net /ISA Bus/A4 renamed /ISA Bus/R_A4
- net /ISA Bus/A5 renamed /ISA Bus/R_A5
- net /ISA Bus/A6 renamed /ISA Bus/R_A6
- net /ISA Bus/A7 renamed /ISA Bus/R_A7
- net /ISA Bus/A8 renamed /ISA Bus/R_A8
- net /ISA Bus/A9 renamed /ISA Bus/R_A9
- net Net-(J1B-~{SMEMR}) renamed /ISA Bus/SMEMR
- J1 pad A1: unconnected-(J1A-D1-PadA1) -> /VL Bus/VL_D1
- J1 pad A10: Net-(J1A-VSS-PadA10) -> GND
- J1 pad A11: unconnected-(J1A-D17-PadA11) -> /VL Bus/VL_D17
- J1 pad A12: Net-(J1A-VCC-PadA12) -> VCC
- J1 pad A13: unconnected-(J1A-D19-PadA13) -> /VL Bus/VL_D19
- J1 pad A14: unconnected-(J1A-D21-PadA14) -> /VL Bus/VL_D21
- J1 pad A15: unconnected-(J1A-D23-PadA15) -> /VL Bus/VL_D23
- J1 pad A16: unconnected-(J1A-D25-PadA16) -> /VL Bus/VL_D25
- J1 pad A17: Net-(J1A-VSS-PadA10) -> GND
- J1 pad A18: unconnected-(J1A-D27-PadA18) -> /VL Bus/VL_D27
- J1 pad A19: unconnected-(J1A-D29-PadA19) -> /VL Bus/VL_D29
- J1 pad A2: unconnected-(J1A-D3-PadA2) -> /VL Bus/VL_D3
- J1 pad A20: unconnected-(J1A-D31-PadA20) -> /VL Bus/VL_D31
- J1 pad A21: unconnected-(J1A-A30-PadA21) -> /VL Bus/VL_A30
- J1 pad A22: unconnected-(J1A-A28-PadA22) -> /VL Bus/VL_A28
- J1 pad A23: unconnected-(J1A-A26-PadA23) -> /VL Bus/VL_A26
- J1 pad A24: Net-(J1A-VSS-PadA10) -> GND
- J1 pad A25: unconnected-(J1A-A24-PadA25) -> /VL Bus/VL_A24
- J1 pad A26: unconnected-(J1A-A22-PadA26) -> /VL Bus/VL_A22
- J1 pad A27: Net-(J1A-VCC-PadA12) -> VCC
- J1 pad A28: unconnected-(J1A-A20-PadA28) -> /VL Bus/VL_A20
- J1 pad A29: unconnected-(J1A-A18-PadA29) -> /VL Bus/VL_A18
- J1 pad A3: Net-(J1A-VSS-PadA10) -> GND
- J1 pad A30: unconnected-(J1A-A16-PadA30) -> /VL Bus/VL_A16
- J1 pad A31: unconnected-(J1A-A14-PadA31) -> /VL Bus/VL_A14
- J1 pad A32: unconnected-(J1A-A12-PadA32) -> /VL Bus/VL_A12
- J1 pad A33: unconnected-(J1A-A10-PadA33) -> /VL Bus/VL_A10
- J1 pad A34: unconnected-(J1A-A8-PadA34) -> /VL Bus/VL_A8
- J1 pad A35: Net-(J1A-VSS-PadA10) -> GND
- J1 pad A36: unconnected-(J1A-A6-PadA36) -> /VL Bus/VL_A6
- J1 pad A37: unconnected-(J1A-A4-PadA37) -> /VL Bus/VL_A4
- J1 pad A39: unconnected-(J1A-BE0-PadA39) -> /VL Bus/BE0
- J1 pad A4: unconnected-(J1A-D5-PadA4) -> /VL Bus/VL_D5
- J1 pad A40: Net-(J1A-VCC-PadA12) -> VCC
- J1 pad A41: unconnected-(J1A-BE1-PadA41) -> /VL Bus/BE1
- J1 pad A42: unconnected-(J1A-BE2-PadA42) -> /VL Bus/BE2
- J1 pad A43: Net-(J1A-VSS-PadA10) -> GND
- J1 pad A44: unconnected-(J1A-BE3-PadA44) -> /VL Bus/BE3
- J1 pad A45: unconnected-(J1A-ADS-PadA45) -> /VL Bus/ADS
- J1 pad A48: unconnected-(J1A-LRDY-PadA48) -> /VL Bus/LRDY
- J1 pad A49: unconnected-(J1A-LDEV-PadA49) -> /VL Bus/LDEV
- J1 pad A5: unconnected-(J1A-D7-PadA5) -> /VL Bus/VL_D7
- J1 pad A50: unconnected-(J1A-LREQ-PadA50) -> /VL Bus/LREQ
- J1 pad A51: Net-(J1A-VSS-PadA10) -> GND
- J1 pad A52: unconnected-(J1A-LGNT-PadA52) -> /VL Bus/LGNT
- J1 pad A53: Net-(J1A-VCC-PadA12) -> VCC
- J1 pad A54: unconnected-(J1A-ID2-PadA54) -> /VL Bus/ID2
- J1 pad A55: unconnected-(J1A-ID3-PadA55) -> /VL Bus/ID3
- J1 pad A56: unconnected-(J1A-ID4-PadA56) -> /VL Bus/ID4
- J1 pad A58: unconnected-(J1A-LEADS-PadA58) -> /VL Bus/LEAD
- J1 pad A6: unconnected-(J1A-D9-PadA6) -> /VL Bus/VL_D9
- J1 pad A7: unconnected-(J1A-D11-PadA7) -> /VL Bus/VL_D11
- J1 pad A8: unconnected-(J1A-D13-PadA8) -> /VL Bus/VL_D13
- J1 pad A9: unconnected-(J1A-D15-PadA9) -> /VL Bus/VL_D15
- J1 pad B1: unconnected-(J1A-D0-PadB1) -> /VL Bus/VL_D0
- J1 pad B10: unconnected-(J1A-D14-PadB10) -> /VL Bus/VL_D14
- J1 pad B11: unconnected-(J1A-D16-PadB11) -> /VL Bus/VL_D16
- J1 pad B12: unconnected-(J1A-D18-PadB12) -> /VL Bus/VL_D18
- J1 pad B13: unconnected-(J1A-D20-PadB13) -> /VL Bus/VL_D20
- J1 pad B14: Net-(J1A-VSS-PadA10) -> GND
- J1 pad B15: unconnected-(J1A-D22-PadB15) -> /VL Bus/VL_D22
- J1 pad B16: unconnected-(J1A-D24-PadB16) -> /VL Bus/VL_D24
- J1 pad B17: unconnected-(J1A-D26-PadB17) -> /VL Bus/VL_D26
- J1 pad B18: unconnected-(J1A-D28-PadB18) -> /VL Bus/VL_D28
- J1 pad B19: unconnected-(J1A-D30-PadB19) -> /VL Bus/VL_D30
- J1 pad B2: unconnected-(J1A-D2-PadB2) -> /VL Bus/VL_D2
- J1 pad B20: Net-(J1A-VCC-PadA12) -> VCC
- J1 pad B21: unconnected-(J1A-A31-PadB21) -> /VL Bus/VL_A31
- J1 pad B22: Net-(J1A-VSS-PadA10) -> GND
- J1 pad B23: unconnected-(J1A-A29-PadB23) -> /VL Bus/VL_A29
- J1 pad B24: unconnected-(J1A-A27-PadB24) -> /VL Bus/VL_A27
- J1 pad B25: unconnected-(J1A-A25-PadB25) -> /VL Bus/VL_A25
- J1 pad B26: unconnected-(J1A-A23-PadB26) -> /VL Bus/VL_A23
- J1 pad B27: unconnected-(J1A-A21-PadB27) -> /VL Bus/VL_A21
- J1 pad B28: unconnected-(J1A-A19-PadB28) -> /VL Bus/VL_A19
- J1 pad B29: Net-(J1A-VSS-PadA10) -> GND
- J1 pad B3: unconnected-(J1A-D4-PadB3) -> /VL Bus/VL_D4
- J1 pad B30: unconnected-(J1A-A17-PadB30) -> /VL Bus/VL_A17
- J1 pad B31: unconnected-(J1A-A15-PadB31) -> /VL Bus/VL_A15
- J1 pad B32: Net-(J1A-VCC-PadA12) -> VCC
- J1 pad B33: unconnected-(J1A-A13-PadB33) -> /VL Bus/VL_A13
- J1 pad B34: unconnected-(J1A-A11-PadB34) -> /VL Bus/VL_A11
- J1 pad B35: unconnected-(J1A-A9-PadB35) -> /VL Bus/VL_A9
- J1 pad B36: unconnected-(J1A-A7-PadB36) -> /VL Bus/VL_A7
- J1 pad B37: unconnected-(J1A-A5-PadB37) -> /VL Bus/VL_A5
- J1 pad B38: Net-(J1A-VSS-PadA10) -> GND
- J1 pad B39: unconnected-(J1A-A3-PadB39) -> /VL Bus/VL_A3
- J1 pad B4: unconnected-(J1A-D6-PadB4) -> /VL Bus/VL_D6
- J1 pad B40: unconnected-(J1A-A2-PadB40) -> /VL Bus/VL_A2
- J1 pad B42: unconnected-(J1A-~{RESET}-PadB42) -> /VL Bus/RST
- J1 pad B44: unconnected-(J1A-M/IO-PadB44) -> /VL Bus/M/IO
- J1 pad B45: unconnected-(J1A-W/R-PadB45) -> /VL Bus/W/R
- J1 pad B48: unconnected-(J1A-RDYRTN-PadB48) -> /VL Bus/RDYR
- J1 pad B49: Net-(J1A-VSS-PadA10) -> GND
- J1 pad B5: unconnected-(J1A-D8-PadB5) -> /VL Bus/VL_D8
- J1 pad B50: unconnected-(J1A-IRQ9-PadB50) -> /VL Bus/IRQ9
- J1 pad B51: unconnected-(J1A-BRDY-PadB51) -> /VL Bus/BRDY
- J1 pad B52: unconnected-(J1A-BLAST-PadB52) -> /VL Bus/BLST
- J1 pad B53: unconnected-(J1A-ID0-PadB53) -> /VL Bus/ID0
- J1 pad B54: unconnected-(J1A-ID1-PadB54) -> /VL Bus/ID1
- J1 pad B55: Net-(J1A-VSS-PadA10) -> GND
- J1 pad B56: unconnected-(J1A-LCLK-PadB56) -> /VL Bus/LCLK
- J1 pad B57: Net-(J1A-VCC-PadA12) -> VCC
- J1 pad B58: unconnected-(J1A-LBS16-PadB58) -> /VL Bus/LBS
- J1 pad B6: Net-(J1A-VSS-PadA10) -> GND
- J1 pad B7: unconnected-(J1A-D10-PadB7) -> /VL Bus/VL_D10
- J1 pad B8: unconnected-(J1A-D12-PadB8) -> /VL Bus/VL_D12
- J1 pad B9: Net-(J1A-VCC-PadA12) -> VCC
- J1 pad C29: +5V -> VCC
- J1 pad C3: +5V -> VCC
- J1 pad C33: /ISA Bus/D7 -> /ISA Bus/ISA_D7
- J1 pad C34: /ISA Bus/D6 -> /ISA Bus/ISA_D6
- J1 pad C35: /ISA Bus/D5 -> /ISA Bus/ISA_D5
- J1 pad C36: /ISA Bus/D4 -> /ISA Bus/ISA_D4
- J1 pad C37: /ISA Bus/D3 -> /ISA Bus/ISA_D3
- J1 pad C38: /ISA Bus/D2 -> /ISA Bus/ISA_D2
- J1 pad C39: /ISA Bus/D1 -> /ISA Bus/ISA_D1
- J1 pad C4: unconnected-(J1B-IRQ2-PadC4) -> /ISA Bus/IRQ2
- J1 pad C40: /ISA Bus/D0 -> /ISA Bus/ISA_D0
- J1 pad C48: /ISA Bus/A14 -> /ISA Bus/R_A14
- J1 pad C7: -12V -> unconnected-(J1B--12V-PadC7)
- U1 pad 1: unconnected-(U1A-SD29-Pad1) -> /VL Bus/VL_D29
- U1 pad 10: unconnected-(U1A-SD23-Pad10) -> /VL Bus/VL_D23
- U1 pad 106: unconnected-(U1C-VCLKI/PD55-Pad106) -> /Memory Bus/PD55
- U1 pad 107: unconnected-(U1C-PD56-Pad107) -> /Memory Bus/PD56
- U1 pad 108: unconnected-(U1C-PD54-Pad108) -> /Memory Bus/PD54
- U1 pad 109: unconnected-(U1C-PD57-Pad109) -> /Memory Bus/PD57
- U1 pad 11: unconnected-(U1A-SD22-Pad11) -> /VL Bus/VL_D22
- U1 pad 110: unconnected-(U1C-PD53-Pad110) -> /Memory Bus/PD53
- U1 pad 111: unconnected-(U1C-PD58-Pad111) -> /Memory Bus/PD58
- U1 pad 112: unconnected-(U1C-PD52-Pad112) -> /Memory Bus/PD52
- U1 pad 113: unconnected-(U1C-PD59-Pad113) -> /Memory Bus/PD59
- U1 pad 115: unconnected-(U1C-PD51-Pad115) -> /Memory Bus/PD51
- U1 pad 116: unconnected-(U1C-PD60-Pad116) -> /Memory Bus/PD60
- U1 pad 117: unconnected-(U1C-PD50-Pad117) -> /Memory Bus/PD50
- U1 pad 118: unconnected-(U1C-PD61-Pad118) -> /Memory Bus/PD61
- U1 pad 119: unconnected-(U1C-PD49-Pad119) -> /Memory Bus/PD49
- U1 pad 12: +5V -> VCC
- U1 pad 120: unconnected-(U1C-PD62-Pad120) -> /Memory Bus/PD62
- U1 pad 121: unconnected-(U1C-PD48-Pad121) -> /Memory Bus/PD48
- U1 pad 122: unconnected-(U1C-PD63-Pad122) -> /Memory Bus/PD63
- U1 pad 124: /Memory Bus/OE -> Net-(U1F-~{OE})
- U1 pad 125: /Memory Bus/WE -> Net-(U1F-~{WE})
- U1 pad 127: unconnected-(U1C-PD39-Pad127) -> /Memory Bus/PD39
- U1 pad 128: unconnected-(U1C-PD40-Pad128) -> /Memory Bus/PD40
- U1 pad 129: unconnected-(U1C-PD38-Pad129) -> /Memory Bus/PD38
- U1 pad 13: unconnected-(U1A-SD21-Pad13) -> /VL Bus/VL_D21
- U1 pad 130: unconnected-(U1C-PD41-Pad130) -> /Memory Bus/PD41
- U1 pad 131: unconnected-(U1C-PD37-Pad131) -> /Memory Bus/PD37
- U1 pad 132: unconnected-(U1C-PD42-Pad132) -> /Memory Bus/PD42
- U1 pad 133: unconnected-(U1C-PD36-Pad133) -> /Memory Bus/PD36
- U1 pad 134: unconnected-(U1C-PD43-Pad134) -> /Memory Bus/PD43
- U1 pad 136: unconnected-(U1C-PD35-Pad136) -> /Memory Bus/PD35
- U1 pad 137: +5V -> VCC
- U1 pad 138: unconnected-(U1C-PD44-Pad138) -> /Memory Bus/PD44
- U1 pad 139: unconnected-(U1C-PD34-Pad139) -> /Memory Bus/PD34
- U1 pad 14: unconnected-(U1A-SD20-Pad14) -> /VL Bus/VL_D20
- U1 pad 140: unconnected-(U1C-PD45-Pad140) -> /Memory Bus/PD45
- U1 pad 141: unconnected-(U1C-PD33-Pad141) -> /Memory Bus/PD33
- U1 pad 142: unconnected-(U1C-PD46-Pad142) -> /Memory Bus/PD46
- U1 pad 143: unconnected-(U1C-PD32-Pad143) -> /Memory Bus/PD32
- U1 pad 144: unconnected-(U1C-PD47-Pad144) -> /Memory Bus/PD47
- U1 pad 146: unconnected-(U1D-LD0/PA0-Pad146) -> Net-(U1D-LD0/PA0)
- U1 pad 147: unconnected-(U1D-LD1/PA1-Pad147) -> Net-(U1D-LD1/PA1)
- U1 pad 148: unconnected-(U1H-LCLK/VCLK-Pad148) -> /LCLK
- U1 pad 149: unconnected-(U1H-HSYNC-Pad149) -> /HS
- U1 pad 15: unconnected-(U1A-SD19-Pad15) -> /VL Bus/VL_D19
- U1 pad 150: unconnected-(U1H-VSYNC-Pad150) -> /VS
- U1 pad 152: /VL Bus/INT -> /VL Bus/SINTR
- U1 pad 153: unconnected-(U1H-~{ROMCS}/GOP1-Pad153) -> /ISA Bus/ROMCS
- U1 pad 154: unconnected-(U1D-LD2/PA2-Pad154) -> Net-(U1D-LD2/PA2)
- U1 pad 155: unconnected-(U1D-LD3/PA3-Pad155) -> Net-(U1D-LD3/PA3)
- U1 pad 156: unconnected-(U1H-XIN-Pad156) -> Net-(U1H-XIN)
- U1 pad 157: unconnected-(U1H-XOUT-Pad157) -> Net-(U1H-XOUT)
- U1 pad 158: +5V -> VCC
- U1 pad 16: unconnected-(U1A-SD18-Pad16) -> /VL Bus/VL_D18
- U1 pad 160: +5V -> VCC
- U1 pad 162: unconnected-(U1H-VREF-Pad162) -> Net-(U1H-VREF)
- U1 pad 164: +5V -> VCC
- U1 pad 166: unconnected-(U1H-RSET-Pad166) -> Net-(U1H-RSET)
- U1 pad 168: unconnected-(U1H-AR-Pad168) -> /S3_RED
- U1 pad 169: +5V -> VCC
- U1 pad 17: unconnected-(U1A-SD17-Pad17) -> /VL Bus/VL_D17
- U1 pad 170: +5V -> VCC
- U1 pad 171: unconnected-(U1H-AG-Pad171) -> /S3_GREEN
- U1 pad 172: unconnected-(U1H-AB-Pad172) -> /S3_BLUE
- U1 pad 174: unconnected-(U1D-LD4/PA4-Pad174) -> Net-(U1D-LD4/PA4)
- U1 pad 175: unconnected-(U1D-LD5/PA5-Pad175) -> Net-(U1D-LD5/PA5)
- U1 pad 176: unconnected-(U1B-SA2-Pad176) -> /VL Bus/VL_A2
- U1 pad 177: unconnected-(U1B-SA3-Pad177) -> /VL Bus/VL_A3
- U1 pad 178: unconnected-(U1B-SA4-Pad178) -> /VL Bus/VL_A4
- U1 pad 179: unconnected-(U1B-SA5-Pad179) -> /VL Bus/VL_A5
- U1 pad 18: unconnected-(U1A-SD16-Pad18) -> /VL Bus/VL_D16
- U1 pad 180: unconnected-(U1B-SA6-Pad180) -> /VL Bus/VL_A6
- U1 pad 181: unconnected-(U1B-SA7-Pad181) -> /VL Bus/VL_A7
- U1 pad 182: unconnected-(U1B-SA8-Pad182) -> /VL Bus/VL_A8
- U1 pad 183: unconnected-(U1B-SA9-Pad183) -> /VL Bus/VL_A9
- U1 pad 184: unconnected-(U1D-LD6/PA6-Pad184) -> Net-(U1D-LD6/PA6)
- U1 pad 185: unconnected-(U1B-SA10-Pad185) -> /VL Bus/VL_A10
- U1 pad 186: unconnected-(U1B-SA11-Pad186) -> /VL Bus/VL_A11
- U1 pad 187: unconnected-(U1B-SA12-Pad187) -> /VL Bus/VL_A12
- U1 pad 188: unconnected-(U1B-SA13-Pad188) -> /VL Bus/VL_A13
- U1 pad 189: unconnected-(U1B-SA14-Pad189) -> /VL Bus/VL_A14
- U1 pad 190: unconnected-(U1B-SA15-Pad190) -> /VL Bus/VL_A15
- U1 pad 191: unconnected-(U1B-SA16-Pad191) -> /VL Bus/VL_A16
- U1 pad 192: +5V -> VCC
- U1 pad 193: /VL Bus/RESET -> Net-(U1G-~{SRESET})
- U1 pad 194: unconnected-(U1G-SCLK-Pad194) -> /VL Bus/LCLK
- U1 pad 196: unconnected-(U1B-SA17-Pad196) -> /VL Bus/VL_A17
- U1 pad 197: unconnected-(U1B-SA18-Pad197) -> /VL Bus/VL_A18
- U1 pad 198: unconnected-(U1B-SA19-Pad198) -> /VL Bus/VL_A19
- U1 pad 199: unconnected-(U1B-SA20-Pad199) -> /VL Bus/VL_A20
- U1 pad 2: unconnected-(U1A-SD28-Pad2) -> /VL Bus/VL_D28
- U1 pad 200: unconnected-(U1B-SA21-Pad200) -> /VL Bus/VL_A21
- U1 pad 201: unconnected-(U1B-SA22-Pad201) -> /VL Bus/VL_A22
- U1 pad 202: unconnected-(U1D-LD7/PA7-Pad202) -> Net-(U1D-LD7/PA7)
- U1 pad 203: unconnected-(U1H-~{VREQ}/VRDY/EVIDEO-Pad203) -> /EVIDEO
- U1 pad 204: unconnected-(U1H-~{CREQ}/CRDY/EVCLK-Pad204) -> /EVCLK
- U1 pad 206: unconnected-(U1H-SPD/~{BLANK}-Pad206) -> /BLANK
- U1 pad 207: unconnected-(U1A-SD31-Pad207) -> /VL Bus/VL_D31
- U1 pad 208: unconnected-(U1A-SD30-Pad208) -> /VL Bus/VL_D30
- U1 pad 21: unconnected-(U1G-~{RDYIN}-Pad21) -> /VL Bus/RDYR
- U1 pad 28: unconnected-(U1A-SD15-Pad28) -> /VL Bus/VL_D15
- U1 pad 29: unconnected-(U1A-SD14-Pad29) -> /VL Bus/VL_D14
- U1 pad 3: unconnected-(U1A-SD27-Pad3) -> /VL Bus/VL_D27
- U1 pad 30: unconnected-(U1A-SD13-Pad30) -> /VL Bus/VL_D13
- U1 pad 31: unconnected-(U1A-SD12-Pad31) -> /VL Bus/VL_D12
- U1 pad 33: unconnected-(U1A-SD11-Pad33) -> /VL Bus/VL_D11
- U1 pad 34: unconnected-(U1A-SD10-Pad34) -> /VL Bus/VL_D10
- U1 pad 35: unconnected-(U1A-SD9-Pad35) -> /VL Bus/VL_D9
- U1 pad 36: unconnected-(U1A-SD8-Pad36) -> /VL Bus/VL_D8
- U1 pad 37: +5V -> VCC
- U1 pad 39: unconnected-(U1A-SD7-Pad39) -> /VL Bus/VL_D7
- U1 pad 4: unconnected-(U1A-SD26-Pad4) -> /VL Bus/VL_D26
- U1 pad 40: unconnected-(U1A-SD6-Pad40) -> /VL Bus/VL_D6
- U1 pad 41: unconnected-(U1A-SD5-Pad41) -> /VL Bus/VL_D5
- U1 pad 42: unconnected-(U1A-SD4-Pad42) -> /VL Bus/VL_D4
- U1 pad 43: unconnected-(U1A-SD3-Pad43) -> /VL Bus/VL_D3
- U1 pad 44: unconnected-(U1A-SD2-Pad44) -> /VL Bus/VL_D2
- U1 pad 45: unconnected-(U1A-SD1-Pad45) -> /VL Bus/VL_D1
- U1 pad 46: unconnected-(U1A-SD0-Pad46) -> /VL Bus/VL_D0
- U1 pad 48: /Memory Bus/CAS4 -> Net-(U1F-~{CAS4})
- U1 pad 49: /Memory Bus/CAS5 -> Net-(U1F-~{CAS5})
- U1 pad 5: unconnected-(U1A-SD25-Pad5) -> /VL Bus/VL_D25
- U1 pad 51: /Memory Bus/CAS6 -> Net-(U1F-~{CAS6})
- U1 pad 52: /Memory Bus/CAS7 -> Net-(U1F-~{CAS7})
- U1 pad 6: unconnected-(U1A-SD24-Pad6) -> /VL Bus/VL_D24
- U1 pad 62: +5V -> VCC
- U1 pad 81: +5V -> VCC
- U1 pad 82: /Memory Bus/CAS3 -> Net-(U1F-~{CAS3})
- U1 pad 83: /Memory Bus/CAS2 -> Net-(U1F-~{CAS2})
- U1 pad 84: /Memory Bus/RAS0 -> Net-(U1F-~{RAS0})
- U1 pad 85: /Memory Bus/CAS1 -> Net-(U1F-~{CAS1})
- U1 pad 86: /Memory Bus/CAS0 -> Net-(U1F-~{CAS0})
- U1 pad 96: +5V -> VCC
- U2 pad 13: /ISA Bus/D0 -> /ISA Bus/R_D7
- U2 pad 14: /ISA Bus/D1 -> /ISA Bus/R_D6
- U2 pad 15: /ISA Bus/D2 -> /ISA Bus/R_D5
- U2 pad 17: /ISA Bus/D3 -> /ISA Bus/R_D4
- U2 pad 18: /ISA Bus/D4 -> /ISA Bus/R_D3
- U2 pad 19: /ISA Bus/D5 -> /ISA Bus/R_D2
- U2 pad 20: /ISA Bus/D6 -> /ISA Bus/R_D1
- U2 pad 21: /ISA Bus/D7 -> /ISA Bus/R_D0
- U2 pad 22: GND -> /ISA Bus/ROMCS
- U5 pad 1: (no net) -> VCC
- U5 pad 10: unconnected-(U5-Pad10) -> /Memory Bus/PD39
- U5 pad 13: unconnected-(U5-Pad13) -> /Memory Bus/WE
- U5 pad 14: unconnected-(U5E-VCC-Pad14) -> /Memory Bus/RAS
- U5 pad 2: (no net) -> /Memory Bus/PD32
- U5 pad 3: (no net) -> /Memory Bus/PD33
- U5 pad 4: unconnected-(U5-Pad4) -> /Memory Bus/PD34
- U5 pad 5: unconnected-(U5-Pad5) -> /Memory Bus/PD35
- U5 pad 6: unconnected-(U5-Pad6) -> VCC
- U5 pad 7: unconnected-(U5E-GND-Pad7) -> /Memory Bus/PD36
- U5 pad 8: unconnected-(U5-Pad8) -> /Memory Bus/PD37
- U5 pad 9: unconnected-(U5-Pad9) -> /Memory Bus/PD38
- U6 pad 1: Net-(R1-Pad2) -> VCC
- U6 pad 10: (no net) -> /Memory Bus/PD55
- U6 pad 11: (no net) -> unconnected-(U6-NC-Pad11)
- U6 pad 12: (no net) -> unconnected-(U6-NC-Pad12)
- U6 pad 13: (no net) -> /Memory Bus/WE
- U6 pad 14: (no net) -> /Memory Bus/RAS
- U6 pad 2: /Memory Bus/RAS0 -> /Memory Bus/PD48
- U6 pad 3: Net-(R2-Pad1) -> /Memory Bus/PD49
- U6 pad 4: (no net) -> /Memory Bus/PD50
- U6 pad 5: (no net) -> /Memory Bus/PD51
- U6 pad 6: (no net) -> VCC
- U6 pad 7: (no net) -> /Memory Bus/PD52
- U6 pad 8: (no net) -> /Memory Bus/PD53
- U6 pad 9: (no net) -> /Memory Bus/PD54
Other:
- board size 240.5 x 121.5 mm -> 338.5 x 121.5 mm
- board text added: "Chamfer 20Deg Edge"

Commit message: PCB work
Parts:
- removed the R1 at (76.0, 82.1)
- removed the R1 at (123.7, 73.0)
- removed the R10 at (144.8, 112.5)
- removed the R10 at (128.1, 84.8)
- removed the R11 at (118.3, 72.5)
- removed the R11 at (144.8, 115.4)
- removed the R2 at (76.0, 85.0)
- removed the R2 at (123.7, 76.0)
- removed the R3 at (76.0, 88.0)
- removed the R3 at (123.7, 79.0)
- removed the R4 at (123.7, 81.9)
- removed the R5 at (76.0, 93.9)
- removed the R5 at (123.7, 84.8)
- removed the R6 at (144.8, 100.7)
- removed the R6 at (128.1, 73.0)
- removed the R7 at (128.1, 76.0)
- removed the R7 at (144.8, 103.6)
- removed the R8 at (128.1, 79.0)
- removed the R8 at (144.8, 106.5)
- removed the R9 at (128.1, 81.9)
- removed the R9 at (144.8, 109.5)
- added FB1: FerriteBead, Inductor_THT:L_Axial_L9.5mm_D4.0mm_P15.24mm_Horizontal_Fastron_SMCC, F.Cu at (262.0, 100.5)
- added FB2: FerriteBead, Inductor_THT:L_Axial_L9.5mm_D4.0mm_P15.24mm_Horizontal_Fastron_SMCC, F.Cu at (262.0, 95.6)
- added FB3: FerriteBead, Inductor_THT:L_Axial_L9.5mm_D4.0mm_P15.24mm_Horizontal_Fastron_SMCC, F.Cu at (262.0, 90.8)
- added G***: LOGO, LOGO, F.Cu at (202.9, 94.2)
- added G***: LOGO, LOGO, F.Cu at (164.5, 85.5)
- added R1: 75R, Resistor_SMD:R_0805_2012Metric_Pad1.20x1.40mm_HandSolder, F.Cu at (240.4, 89.8)
- added R10: 33R, Resistor_SMD:R_0805_2012Metric_Pad1.20x1.40mm_HandSolder, F.Cu at (150.4, 133.9)
- added R11: 33R, Resistor_SMD:R_0805_2012Metric_Pad1.20x1.40mm_HandSolder, F.Cu at (174.9, 114.2)
- added R2: 75R, Resistor_SMD:R_0805_2012Metric_Pad1.20x1.40mm_HandSolder, F.Cu at (240.4, 94.6)
- added R3: 75R, Resistor_SMD:R_0805_2012Metric_Pad1.20x1.40mm_HandSolder, F.Cu at (240.4, 99.4)
- added R34: 10K, Resistor_SMD:R_0805_2012Metric_Pad1.20x1.40mm_HandSolder, F.Cu at (88.9, 108.3)
- added R5: 33R, Resistor_SMD:R_0805_2012Metric_Pad1.20x1.40mm_HandSolder, F.Cu at (259.0, 105.8)
- added R6: 33R, Resistor_SMD:R_0805_2012Metric_Pad1.20x1.40mm_HandSolder, F.Cu at (122.3, 73.3)
- added R7: 33R, Resistor_SMD:R_0805_2012Metric_Pad1.20x1.40mm_HandSolder, F.Cu at (127.0, 72.8)
- added R8: 33R, Resistor_SMD:R_0805_2012Metric_Pad1.20x1.40mm_HandSolder, F.Cu at (128.5, 131.1)
- added R9: 33R, Resistor_SMD:R_0805_2012Metric_Pad1.20x1.40mm_HandSolder, F.Cu at (155.1, 133.2)
- U1: value 86C375 -> 86C325
- U10: value 74F245 -> 74LS245; footprint Package_SO:SO-20_5.3x12.6mm_P1.27mm -> Package_DIP:DIP-20_W7.62mm
- moved JP2 184.6 mm to (53.0, 126.7)
- moved C9 171.3 mm to (88.9, 106.3), turned to 180 degrees
- moved C1 167.5 mm to (242.8, 89.8), turned to 90 degrees
- moved C2 167.4 mm to (242.8, 94.6), turned to 90 degrees
- moved JP1 91.2 mm to (267.8, 112.4)
- moved U5 86.5 mm to (82.5, 86.0), turned to 90 degrees
- moved R17 79.4 mm to (66.8, 135.4), turned to -90 degrees
- moved U6 65.2 mm to (117.3, 86.0), turned to 90 degrees
- moved R14 53.9 mm to (107.1, 73.4)
- moved R13 44.7 mm to (115.1, 75.2)
- moved C3 39.0 mm to (242.8, 99.4), turned to 90 degrees
- moved R23 37.6 mm to (55.5, 91.8), turned to 180 degrees
- moved R30 36.8 mm to (55.5, 101.9)
- moved U2 32.4 mm to (226.9, 116.8)
- moved R31 31.7 mm to (55.5, 104.1), turned to 180 degrees
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Connections:
- J1 pad A50: /VL Bus/LREQ -> unconnected-(J1A-LREQ-PadA50)
- J1 pad A52: /VL Bus/LGNT -> unconnected-(J1A-LGNT-PadA52)
- J1 pad A58: /VL Bus/LEAD -> unconnected-(J1A-LEADS-PadA58)
- J1 pad B51: /VL Bus/BRDY -> unconnected-(J1A-BRDY-PadB51)
- J1 pad B52: /VL Bus/BLST -> unconnected-(J1A-BLAST-PadB52)
- J1 pad B58: /VL Bus/LBS -> unconnected-(J1A-LBS16-PadB58)
- R28 pad 2: unconnected-(R28-Pad2) -> /ESYNC
- U1 pad 165: unconnected-(U1H-~{PDOWN}-Pad165) -> Net-(U1H-~{PDOWN})
- U1 pad 205: unconnected-(U1H-SPCLK/ESYNC-Pad205) -> /ESYNC
- U1 pad 23: unconnected-(U1G-~{SRDY}-Pad23) -> /VL Bus/LRDY
- U1 pad 24: unconnected-(U1G-~{LOCA}-Pad24) -> /VL Bus/LDEV
- U2 pad 13: /ISA Bus/R_D7 -> /ISA Bus/R_D0
- U2 pad 14: /ISA Bus/R_D6 -> /ISA Bus/R_D1
- U2 pad 15: /ISA Bus/R_D5 -> /ISA Bus/R_D2
- U2 pad 17: /ISA Bus/R_D4 -> /ISA Bus/R_D3
- U2 pad 18: /ISA Bus/R_D3 -> /ISA Bus/R_D4
- U2 pad 19: /ISA Bus/R_D2 -> /ISA Bus/R_D5
- U2 pad 20: /ISA Bus/R_D1 -> /ISA Bus/R_D6
- U2 pad 21: /ISA Bus/R_D0 -> /ISA Bus/R_D7
Routing:
- net /VS: track 0.00 -> 254.9 mm, vias 0 -> 1
- net /HS: track 0.00 -> 235.3 mm, vias 0 -> 1
- net /Memory Bus/MA3: track 0.00 -> 158.1 mm, vias 0 -> 5
- net /Memory Bus/MA4: track 0.00 -> 157.2 mm, vias 0 -> 5
- net /Memory Bus/MA5: track 0.00 -> 154.7 mm, vias 0 -> 5
- net /Memory Bus/MA2: track 0.00 -> 154.0 mm, vias 0 -> 5
- net /Memory Bus/MA1: track 0.00 -> 152.1 mm, vias 0 -> 5
- net /Memory Bus/MA6: track 0.00 -> 151.3 mm, vias 0 -> 5
- net /Memory Bus/MA7: track 0.00 -> 150.8 mm, vias 0 -> 5
- net /Memory Bus/MA0: track 0.00 -> 148.7 mm, vias 0 -> 5
- net /Memory Bus/MA8: track 0.00 -> 145.6 mm, vias 0 -> 5
- net /ISA Bus/ROMCS: track 0.00 -> 124.0 mm, vias 0 -> 1
- net /VL Bus/SINTR: track 0.00 -> 81.9 mm, vias 0 -> 1
- net /ESYNC: track 0.00 -> 69.2 mm, vias 0 -> 2
- net /EVIDEO: track 0.00 -> 69.0 mm, vias 0 -> 2
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- added copper zone on F.Cu, net GND
Other:
- board size 338.5 x 121.5 mm -> 240.5 x 70.4 mm
- copper layers 2 -> 4
- board text added: "86C325 (ViRGE)"
- board text added: "86C765 (Trio 64V+)"
- board text added: "or"
- board text removed: "Chamfer 20Deg Edge"

Commit message: even more PCB work
Parts:
- removed G*** (x2): LOGO, LOGO
- added ?: , clipboard:1487c8fc-82e6-4f6f-bb8e-5a80aa76ea0e, F.Cu at (199.9, 99.3)
- added ?: , clipboard:13d0430b-84c4-4042-9416-d42f9d9306b6, F.Cu at (158.1, 90.0)
- FB1, FB2, FB3: footprint Inductor_THT:L_Axial_L9.5mm_D4.0mm_P15.24mm_Horizontal_Fastron_SMCC -> Inductor_SMD:L_0805_2012Metric_Pad1.15x1.40mm_HandSolder
- moved R14 46.5 mm to (153.0, 80.1), turned to 90 degrees
- moved R13 41.3 mm to (156.1, 80.1), turned to 90 degrees
- moved R7 29.5 mm to (111.4, 97.8)
- moved R6 26.1 mm to (113.4, 97.8)
- moved R3 18.5 mm to (258.7, 102.4), turned to -90 degrees
- moved R1 15.3 mm to (255.5, 92.5)
- moved R8 14.4 mm to (142.9, 131.3)
- moved R2 14.1 mm to (254.1, 97.9), turned to -90 degrees
- moved C3 13.8 mm to (256.3, 102.4), turned to -90 degrees
- moved C1 10.8 mm to (253.2, 92.5)
- moved JP2 9.88 mm to (49.5, 117.5)
- moved C2 9.48 mm to (251.7, 97.9), turned to -90 degrees
- moved JP1 8.57 mm to (273.3, 119.0), turned to 90 degrees
- moved FB3 7.57 mm to (259.1, 97.8)
- moved FB1 7.46 mm to (259.1, 93.6)
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Connections:
- FB1 pad 1: /BLUE -> /RED
- FB1 pad 2: /S3_BLUE -> /S3_RED
- FB3 pad 1: /RED -> /BLUE
- FB3 pad 2: /S3_RED -> /S3_BLUE
Routing:
- net /S3_BLUE: track 6.38 -> 196.6 mm
- net GND: track 0.00 -> 186.0 mm, vias 0 -> 53
- net /S3_GREEN: track 6.38 -> 188.0 mm
- net /S3_RED: track 2.43 -> 182.6 mm
- net Net-(U1F-~{CAS5}): track 0.00 -> 107.7 mm, vias 0 -> 2
- net Net-(U1F-~{CAS4}): track 0.00 -> 103.9 mm, vias 0 -> 2
- net Net-(U1F-~{CAS6}): track 0.00 -> 99.3 mm, vias 0 -> 2
- net VCC: track 0.00 -> 99.1 mm, vias 0 -> 31
- net Net-(U1F-~{CAS7}): track 0.00 -> 97.5 mm, vias 0 -> 2
- net /BLANK: track 0.00 -> 85.3 mm, vias 0 -> 2
- net /ISA Bus/SMEMR: track 0.00 -> 78.8 mm
- net /Memory Bus/WE: track 0.00 -> 62.6 mm
- net /Memory Bus/OE: track 0.00 -> 60.4 mm
- net /ISA Bus/ROMCS: track 124.0 -> 182.7 mm
- net /Memory Bus/CAS4: track 0.00 -> 58.1 mm
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- added copper zone on In1.Cu, net GND
- added copper zone on In2.Cu, net VCC
- removed copper zone on F.Cu, net GND
