File: files/virge-vlb.kicad_pcb (KiCad board)
At the start: 4 copper layers, 240.5 x 70.4 mm, 94 parts, among them J1 VLB_slot, J2 VGA, U1 86C325, U10 7408, U2 27C020, U7 74LS244, U8 4052, U9 7404, Y1 14.318MHz

Commit message: final touches
Parts:
- C5, C8: value 10pF -> 3 x 10pF
- R10, R13: value 33R -> 3 x 33R
- R16, R6: value 33R -> 2 x 33R
- R44: value 10K -> 10K each
- R5: value 75R -> 3 x 75R
- moved C15 15.3 mm to (47.6, 129.0), turned to 180 degrees
- moved C1 14.3 mm to (252.7, 118.5)
- moved C10 14.3 mm to (117.1, 123.2)
- moved C14 14.3 mm to (230.1, 130.5)
- moved C2 14.3 mm to (252.7, 116.0)
- moved C21 14.3 mm to (171.4, 129.5)
- moved C22 14.3 mm to (247.6, 129.5)
- moved C3 14.3 mm to (252.9, 86.0)
- moved C5 14.3 mm to (244.6, 86.0)
- moved C6 14.3 mm to (252.7, 96.3)
- moved C8 14.3 mm to (244.6, 96.3)
- moved R1 14.3 mm to (252.7, 120.7)
- moved R13 14.3 mm to (143.1, 78.8)
- moved R3 14.3 mm to (252.9, 88.3)
- moved R38 14.3 mm to (160.5, 104.6)
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Routing:
- net GND: track 178.0 -> 178.4 mm, vias 170 -> 187
Other:
- rule pad_to_mask_clearance: 0 -> 0.038
- rule solder_mask_min_width: 0.12 -> 0.13
- board text added: "(install R54 if 28 pin is used)"
- board text added: "0xCats (PCB)"
- board text added: "27C010"
- board text added: "People who helped make this card:"
- board text added: "Rev 1.0"
- board text added: "VREF"
- board text added: "Video BIOS 27C256/512"
- board text added: "computerguy096 (PCB)"
- board text added: "limsup (art design)"
- board text removed: "VREF adj."
- board text removed: "Video BIOS"
