File: files/virge-vlb.kicad_pcb (KiCad board)
At the start: 4 copper layers, 240.5 x 70.4 mm, 94 parts, among them J1 VLB_slot, J2 VGA, U1 86C325, U10 7408, U2 27C020, U7 74LS244, U8 4052, U9 7404, Y1 14.318MHz

Commit message: Board review changes 2023-07-06
Parts:
- removed C16: 0.1uF, Capacitor_SMD:C_0805_2012Metric_Pad1.18x1.45mm_HandSolder
- removed U8: 4052, Package_SO:SO-16_3.9x9.9mm_P1.27mm
- C5, C8: value 3 x 10pF -> 10pF
- R10, R13: value 3 x 33R -> 33R
- R16, R6: value 2 x 33R -> 33R
- R19, R20: value 10K -> 0
- R21: value 4K7 -> 4.7K
- R44: value 10K each -> 10K
- R5: value 3 x 75R -> 75R
- moved R19 121.8 mm to (173.9, 120.8)
- moved R21 118.8 mm to (174.9, 123.8), turned to 180 degrees
- moved R20 117.5 mm to (171.8, 120.8)
- moved R18 112.0 mm to (170.8, 123.8)
- moved C18 104.4 mm to (176.2, 120.8)
- moved C17 100.0 mm to (169.6, 120.8)
- moved JP1 3.96 mm to (243.0, 105.5)
- moved C11 3.20 mm to (144.6, 129.6)
- moved R55 2.66 mm to (229.2, 120.0)
- moved C19 1.69 mm to (130.4, 132.4)
Connections:
- net /ISA Bus/ROMCS renamed ROMCS
- net Net-(C1-Pad1) renamed /HS_VGA
- net Net-(C2-Pad1) renamed /VS_VGA
- net Net-(U10-Pad1) renamed /VL Bus/VL_A23_O
- net Net-(U10-Pad10) renamed /VL Bus/VL_A25+A26
- net Net-(U10-Pad12) renamed /VL Bus/VL_A23-A26
- net Net-(U10-Pad13) renamed /VL Bus/VL_A29_O
- net Net-(U10-Pad2) renamed /VL Bus/VL_A24_O
- net Net-(U10-Pad3) renamed /VL Bus/VL_A23+A24
- net Net-(U10-Pad4) renamed /VL Bus/VL_A25_O
- net Net-(U10-Pad5) renamed /VL Bus/VL_A26_O
- C17 pad 1: /DDC_SDA -> GND
- C17 pad 2: GND -> /DDC_SDA
- C18 pad 1: /DDC_SCL -> GND
- C18 pad 2: GND -> /DDC_SCL
- R18 pad 2: Net-(U8-X1) -> /SPD
- R19 pad 1: Net-(U8-Y1) -> /SPCLK
- R19 pad 2: VCC -> /DDC_SCL
- R20 pad 1: VCC -> /DDC_SDA
- R20 pad 2: /DDC_SDA -> /SPD
- R21 pad 2: /DDC_SCL -> /SPCLK
- U1 pad 151: /ENFEAT -> unconnected-(U1H-~{GPIOSTR}/~{ENFEAT}/GOP0-Pad151)
- U9 pad 9: GND -> VCC
Routing:
- net /DDC_SDA: track 284.2 -> 104.5 mm
- net /DDC_SCL: track 264.2 -> 100.1 mm
- net /SPCLK: track 43.1 -> 112.3 mm
- net /SPD: track 43.8 -> 109.8 mm
- net /ENFEAT: track 46.3 -> 0.00 mm
- net VCC: track 172.2 -> 148.4 mm, vias 37 -> 44
- net Net-(U8-Y1): track 16.9 -> 0.00 mm
- net GND: track 178.4 -> 162.3 mm, vias 187 -> 203
- net Net-(U8-B): track 8.47 -> 0.00 mm
- net /VS: track 190.4 -> 185.4 mm
- net Net-(U8-X1): track 4.52 -> 0.00 mm
- net Net-(JP1-Pin_2): track 16.6 -> 20.7 mm
- net ROMCS: track 186.7 -> 189.5 mm
- net /ISA Bus/R_A12: track 39.2 -> 36.3 mm
- net /HS: track 193.3 -> 190.6 mm
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- added copper zone on F.Cu, net (none)
- added copper zone on In1.Cu, net (none)
- added copper zone on In2.Cu, net (none)

Commit message: fixed some clearance issues, fixed S3 logo, fixed annotations
Parts:
- removed the C14 at (230.1, 130.5)
- removed the C17 at (169.6, 120.8)
- removed the C18 at (176.2, 120.8)
- removed the R19 at (173.9, 120.8)
- removed the R20 at (171.8, 120.8)
- removed the U9 at (124.2, 132.2)
- added C9: 100nF, Capacitor_SMD:C_0805_2012Metric_Pad1.18x1.45mm_HandSolder, F.Cu at (232.2, 130.9)
- added R8: 4.7K, Resistor_SMD:R_0805_2012Metric_Pad1.20x1.40mm_HandSolder, F.Cu at (176.2, 120.0)
- added R9: 33R, Resistor_SMD:R_0805_2012Metric_Pad1.20x1.40mm_HandSolder, F.Cu at (172.4, 120.0)
- added U8: 7404, Package_SO:SO-14_3.9x8.65mm_P1.27mm, F.Cu at (124.2, 132.2)
- R13: renamed from R10; value 33R -> 3 x 33R
- R23: renamed from R44; value 10K -> 10K each
- moved C22 4.17 mm to (51.5, 121.3)
- moved R10 2.38 mm to (172.4, 122.1)
- moved R11 2.17 mm to (176.2, 122.1)
- moved R6 1.76 mm to (230.5, 118.8), turned to 0 degrees
- moved R44 1.35 mm to (52.2, 133.7), turned to -90 degrees
- moved C13 1.14 mm to (66.8, 87.8)
- moved C14 1.02 mm to (73.7, 103.7)
- moved R43 1.02 mm to (73.7, 105.7)
- turned C12 to -90 degrees
- renumbered C9 to C14, C28 to C16, C27 to C17, C20 to C18, C22 to C20, C23 to C22, C24 to C23, C25 to C24, C26 to C25, R18 to R10, R21 to R11, R9 to R12, R11 to R14, R12 to R15, R13 to R16, R14 to R17, R15 to R18, R16 to R19, R8 to R20, R7 to R21, R6 to R22, R43 to R24, R39 to R25, R40 to R26, R41 to R27, R42 to R28, R37 to R29, R38 to R30, R45 to R31, R46 to R32, R47 to R33, R53 to R34, R48 to R35, R52 to R36, R51 to R37, R50 to R38, R49 to R39, R36 to R40, R35 to R41, R33 to R42, R34 to R43, R17 to R44, R24 to R45, R22 to R46, R23 to R47, R55 to R6, R54 to R7, U7 to U1, U1 to U7, U10 to U9
Connections:
- C12 pad 1: VCC -> GND
- C12 pad 2: GND -> VCC
- J2 pad 12: /DDC_SDA -> /DDC_SDA_VGA
- J2 pad 15: /DDC_SCL -> /DDC_SCL_VGA
- R10 pad 2: /SPD -> /DDC_SDA
- R11 pad 2: /SPCLK -> /DDC_SCL
- U7 pad 205: /SPCLK -> /DDC_SCL
- U7 pad 206: /SPD -> /DDC_SDA
Routing:
- net /SPCLK: track 112.3 -> 0.00 mm, vias 2 -> 0
- net /SPD: track 109.8 -> 0.00 mm, vias 2 -> 0
- net /DDC_SDA_VGA: track 0.00 -> 101.9 mm, vias 0 -> 1
- net /DDC_SCL_VGA: track 0.00 -> 94.6 mm, vias 0 -> 1
- net /VL Bus/ADS: track 69.7 -> 101.0 mm
- net /DDC_SCL: track 100.1 -> 113.8 mm, vias 1 -> 2
- net GND: track 162.3 -> 153.6 mm, vias 203 -> 204
- net VCC: track 148.4 -> 140.1 mm, vias 44 -> 46
- net /DDC_SDA: track 104.5 -> 111.6 mm, vias 1 -> 2
- net /VL Bus/LDEV: track 75.8 -> 81.4 mm
- net /VL Bus/VL_A5: track 42.8 -> 45.6 mm
- net /VL Bus/BE2: track 62.2 -> 64.9 mm
- net /VL Bus/VL_A17: track 29.8 -> 27.2 mm
- net /VL Bus/W/R: track 68.5 -> 71.0 mm
- net /Memory Bus/MA3: track 160.5 -> 158.2 mm
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- removed copper zone on In1.Cu, net (none)
- removed copper zone on In2.Cu, net (none)

Commit message: final changes for revision 1A
Parts:
- added R48: 33R, Resistor_SMD:R_0805_2012Metric_Pad1.20x1.40mm_HandSolder, F.Cu at (255.9, 108.3)
- JP1: value Conn_01x02 -> DDC 5V
- moved JP1 7.08 mm to (249.4, 108.3), turned to 90 degrees
- moved C12 0.35 mm to (138.9, 79.1)
Connections:
- J2 pad 9: Net-(JP1-Pin_2) -> Net-(J2-Pad9)
Routing:
- net Net-(JP1-Pin_2): track 20.7 -> 2.95 mm
- net VCC: track 140.1 -> 128.9 mm
- net GND: track 153.6 -> 162.6 mm
- net Net-(J2-Pad9): track 0.00 -> 6.75 mm
- removed copper zone on F.Cu, net (none)
Other:
- board size 240.5 x 70.4 mm -> 240.5 x 69.4 mm
- board text added: "JLCJLCJLCJLC"
- board text added: "Rev 1A"
- board text added: "Special thanks to:"
- board text added: "by computerguy096"
- board text removed: "People who helped make this card:"
- board text removed: "Rev 1.0"
- board text removed: "computerguy096 (PCB)"
