File: files/busctrl.kicad_sch (KiCad schematic)
At the start: 5 parts, among them J1 VLB_slot, U2 27C020, U7 74LS244

Commit message: fixed some clearance issues, fixed S3 logo, fixed annotations
Parts:
- added C14: 100nF, Capacitor_SMD:C_0805_2012Metric_Pad1.18x1.45mm_HandSolder, symbol Device:C
- renumbered U7 to U1
Connections:
- net GND: now also C14.2
- net VCC: now also C14.1
Changed lines of the file:
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@@
   (junction (at 57.15 95.25) (diameter 0) (color 0 0 0 0)
+  )
+  (junction (at 69.85 53.34) (diameter 0) (color 0 0 0 0)
   )
   (no_connect (at 157.48 134.62))
@@
     (stroke (width 0) (type default))
   )
+  (wire (pts (xy 55.88 53.34) (xy 69.85 53.34))
+    (stroke (width 0) (type default))
+  )
   (wire (pts (xy 102.87 77.47) (xy 109.22 77.47))
     (stroke (width 0) (type default))
@@
   )
   (wire (pts (xy 102.87 90.17) (xy 109.22 90.17))
+    (stroke (width 0) (type default))
+  )
+  (wire (pts (xy 69.85 53.34) (xy 69.85 62.23))
     (stroke (width 0) (type default))
   )
@@
     )
   )
+  (symbol (lib_id "power:GND") (at 55.88 60.96 0) (unit 1)
+    (in_bom yes) (on_board yes) (dnp no)
+    (property "Reference" "#PWR024" (at 55.88 67.31 0)
+      (effects (font (size 1.27 1.27)) hide)
+    )
+    (property "Value" "GND" (at 53.34 64.77 0)
+      (effects (font (size 1.27 1.27)))
+    )
+    (property "Footprint" "" (at 55.88 60.96 0)
+      (effects (font (size 1.27 1.27)) hide)
+    )
+    (property "Datasheet" "" (at 55.88 60.96 0)
+      (effects (font (size 1.27 1.27)) hide)
+    )
+    (pin "1")
+    (instances
+      (project "virge-vlb"
+        (path "/e8216711-86b5-4276-82f4-4c7ed22b9a9c/485e825d-a3d2-4e3d-9ea7-d005dd511bf5"
+          (reference "#PWR024") (unit 1)
+        )
+        (path "/e8216711-86b5-4276-82f4-4c7ed22b9a9c/9321f466-5ac6-411a-b039-07fb7f0cdeaa"
+          (reference "#PWR024") (unit 1)
+        )
+      )
+    )
+  )
   (symbol (lib_id "Device:R") (at 96.52 107.95 270) (unit 1)
     (in_bom yes) (on_board yes) (dnp no)
@@
         )
         (path "/e8216711-86b5-4276-82f4-4c7ed22b9a9c/485e825d-a3d2-4e3d-9ea7-d005dd511bf5"
-          (reference "R55") (unit 1)
+          (reference "R6") (unit 1)
         )
       )
@@
   (symbol (lib_id "74xx:74LS244") (at 69.85 82.55 0) (unit 1)
     (in_bom yes) (on_board yes) (dnp no) (fields_autoplaced)
-    (property "Reference" "U7" (at 71.8059 63.5 0)
+    (property "Reference" "U1" (at 71.8059 63.5 0)
       (effects (font (size 1.27 1.27)) (justify left))
     )
@@
       (project "virge-vlb"
         (path "/e8216711-86b5-4276-82f4-4c7ed22b9a9c/485e825d-a3d2-4e3d-9ea7-d005dd511bf5"
-          (reference "U7") (unit 1)
-        )
-      )
-    )
-  )
-  (symbol (lib_id "power:VCC") (at 69.85 62.23 0) (unit 1)
+          (reference "U1") (unit 1)
+        )
+      )
+    )
+  )
+  (symbol (lib_id "power:VCC") (at 69.85 53.34 0) (unit 1)
     (in_bom yes) (on_board yes) (dnp no) (fields_autoplaced)
-    (property "Reference" "#PWR026" (at 69.85 66.04 0)
-      (effects (font (size 1.27 1.27)) hide)
-    )
-    (property "Value" "VCC" (at 69.85 58.42 0)
+    (property "Reference" "#PWR026" (at 69.85 57.15 0)
+      (effects (font (size 1.27 1.27)) hide)
+    )
+    (property "Value" "VCC" (at 69.85 49.53 0)
       (effects (font (size 1.27 1.27)))
     )
-    (property "Footprint" "" (at 69.85 62.23 0)
-      (effects (font (size 1.27 1.27)) hide)
-    )
-    (property "Datasheet" "" (at 69.85 62.23 0)
+    (property "Footprint" "" (at 69.85 53.34 0)
+      (effects (font (size 1.27 1.27)) hide)
+    )
+    (property "Datasheet" "" (at 69.85 53.34 0)
       (effects (font (size 1.27 1.27)) hide)
     )
@@
     )
   )
+  (symbol (lib_id "Device:C") (at 55.88 57.15 0) (unit 1)
+    (in_bom yes) (on_board yes) (dnp no)
+    (property "Reference" "C14" (at 58.42 55.88 0)
+      (effects (font (size 1.27 1.27)) (justify left))
+    )
+    (property "Value" "100nF" (at 58.42 59.69 0)
+      (effects (font (size 1.27 1.27)) (justify left))
+    )
+    (property "Footprint" "Capacitor_SMD:C_0805_2012Metric_Pad1.18x1.45mm_HandSolder" (at 56.8452 60.96 0)
+      (effects (font (size 1.27 1.27)) hide)
+    )
+    (property "Datasheet" "~" (at 55.88 57.15 0)
+      (effects (font (size 1.27 1.27)) hide)
+    )
+    (pin "1")
+    (pin "2")
+    (instances
+      (project "virge-vlb"
+        (path "/e8216711-86b5-4276-82f4-4c7ed22b9a9c"
+          (reference "C14") (unit 1)
+        )
+        (path "/e8216711-86b5-4276-82f4-4c7ed22b9a9c/485e825d-a3d2-4e3d-9ea7-d005dd511bf5"
+          (reference "C9") (unit 1)
+        )
+      )
+    )
+  )
   (symbol (lib_id "power:GND") (at 69.85 102.87 0) (unit 1)
     (in_bom yes) (on_board yes) (dnp no) (fields_autoplaced)
@@
         )
         (path "/e8216711-86b5-4276-82f4-4c7ed22b9a9c/485e825d-a3d2-4e3d-9ea7-d005dd511bf5"
-          (reference "R54") (unit 1)
-        )
-      )
+          (reference "R7") (unit 1)
+        )
+      )
