File: files/virge-vlb.kicad_sch (KiCad schematic)
At the start: 48 parts, among them J2 VGA, U1 86C325, U8 4052, U9 7404, Y1 14.318MHz

Commit message: Board review changes 2023-07-06
Parts:
- removed C16: 0.1uF, Capacitor_SMD:C_0805_2012Metric_Pad1.18x1.45mm_HandSolder, symbol Device:C
- removed C19, C20: 100nF, Capacitor_SMD:C_0805_2012Metric_Pad1.18x1.45mm_HandSolder, symbol Device:C
- removed R19, R20: 10K, Resistor_SMD:R_0805_2012Metric_Pad1.20x1.40mm_HandSolder, symbol Device:R
- removed U8: 4052, Package_SO:SO-16_3.9x9.9mm_P1.27mm, symbol 4xxx:4052
- added R19, R20: 0, Resistor_SMD:R_0805_2012Metric_Pad1.20x1.40mm_HandSolder, symbol Device:R_Small
- JP1: Function (none) -> SPI Power DDC/i2c ROM
- R21: value 4K7 -> 4.7K
Connections:
- net DDC_SCL: now also C18.2, R19.2; no longer C18.1, R21.2
- net DDC_SDA: now also C17.2, R20.1; no longer C17.1
- net GND: now also C17.1, C18.1; no longer C17.2, C18.2
- net SPCLK: now also R21.2, R19.1
- net SPD: now also R18.2, R20.2
- net VS_VGA: now reaches C2.1, J2.14, R2.2
- net HS_VGA: now reaches C1.1, J2.13, R1.2
- net ENFEAT: no longer names the net of U1.151 (~{GPIOSTR}/~{ENFEAT}/GOP0)
- net ISA Bus/ROMCS renamed ROMCS
- no-connect marks 15 -> 14
Other:
- sheet ISA Bus ports: added none; removed ROMCS
- note added: "NO STUFF C18,C17 Test if needed"
- note added: "TODO"
- moved on the sheet: C1, C17, C18, C2, C3, C4, C5, C6, C7, C8, FB1, FB2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

Commit message: fixed some clearance issues, fixed S3 logo, fixed annotations
Parts:
- removed C10, C11, C12, C13, C14: 100nF, Capacitor_SMD:C_0805_2012Metric_Pad1.18x1.45mm_HandSolder, symbol Device:C
- removed C17, C18: 0.1uF, Capacitor_SMD:C_0805_2012Metric_Pad1.18x1.45mm_HandSolder, symbol Device:C
- removed R19, R20: 0, Resistor_SMD:R_0805_2012Metric_Pad1.20x1.40mm_HandSolder, symbol Device:R_Small
- removed U9: 7404, Package_SO:SO-14_3.9x8.65mm_P1.27mm, symbol 74xx:74HC04
- added R8: 4.7K, Resistor_SMD:R_0805_2012Metric_Pad1.20x1.40mm_HandSolder, symbol Device:R
- added R9: 33R, Resistor_SMD:R_0805_2012Metric_Pad1.20x1.40mm_HandSolder, symbol Device:R
- renumbered C9 to C14, C28 to C16, C27 to C17, C22 to C20, C23 to C22, C24 to C23, C25 to C24, C26 to C25, R18 to R10, R21 to R11, R35 to R41, R33 to R42, R34 to R43
Connections:
- net SPCLK is gone; now on net DDC_SCL: R11.2, U1.205 (SPCLK/ESYNC)
- net SPD is gone; now on net DDC_SDA: R10.2, U1.206 (SPD/~{BLANK})
- net DDC_SCL: now also R8.1; no longer J2.15
- net DDC_SDA: now also R9.1; no longer J2.12
- new net DDC_SCL_VGA: J2.15, R8.2
- new net DDC_SDA_VGA: J2.12, R9.2
Other:
- note removed: "NO STUFF C18,C17 Test if needed"
- moved on the sheet: C1, C2, C20, C21, C22, C23, C24, C25, R10, R11

Commit message: final changes for revision 1A
Parts:
- added R48: 33R, Resistor_SMD:R_0805_2012Metric_Pad1.20x1.40mm_HandSolder, symbol Device:R
- JP1: value Conn_01x02 -> DDC 5V
Connections:
- net at JP1.2 (Pin_2): now also R48.2; no longer J2.9
- new net: J2.9, R48.1
Other:
- moved on the sheet: JP1
Changed lines of the file:
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@@
+    (stroke (width 0) (type default))
+  )
+  (wire (pts (xy 78.74 148.59) (xy 85.09 148.59))
     (stroke (width 0) (type default))
   )
@@
     (stroke (width 0) (type default))
   )
-  (wire (pts (xy 78.74 148.59) (xy 90.17 148.59))
-    (stroke (width 0) (type default))
-  )
   (wire (pts (xy 40.64 151.13) (xy 63.5 151.13))
     (stroke (width 0) (type default))
@@
     (stroke (width 0) (type default))
   )
-  (wire (pts (xy 90.17 146.05) (xy 88.9 146.05))
+  (wire (pts (xy 99.06 144.78) (xy 97.79 144.78))
     (stroke (width 0) (type default))
   )
@@
     (stroke (width 0) (type default))
   )
+  (wire (pts (xy 85.09 148.59) (xy 85.09 147.32))
+    (stroke (width 0) (type default))
+  )
   (wire (pts (xy 83.82 143.51) (xy 78.74 143.51))
     (stroke (width 0) (type default))
@@
     (stroke (width 0) (type default))
   )
-  (wire (pts (xy 88.9 146.05) (xy 88.9 143.51))
+  (wire (pts (xy 97.79 144.78) (xy 97.79 142.24))
     (stroke (width 0) (type default))
   )
@@
   )
   (wire (pts (xy 153.67 170.18) (xy 158.75 170.18))
+    (stroke (width 0) (type default))
+  )
+  (wire (pts (xy 85.09 147.32) (xy 91.44 147.32))
     (stroke (width 0) (type default))
   )
@@
     )
   )
-  (symbol (lib_id "Connector_Generic:Conn_01x02") (at 95.25 146.05 0) (unit 1)
-    (in_bom yes) (on_board yes) (dnp no)
-    (property "Reference" "JP1" (at 97.79 147.32 0)
-      (effects (font (size 1.27 1.27)) (justify left))
-    )
-    (property "Value" "Conn_01x02" (at 97.79 149.225 0)
-      (effects (font (size 1.27 1.27)) (justify left) hide)
-    )
-    (property "Footprint" "Connector_PinHeader_2.54mm:PinHeader_1x02_P2.54mm_Vertical" (at 95.25 146.05 0)
-      (effects (font (size 1.27 1.27)) hide)
-    )
-    (property "Datasheet" "~" (at 95.25 146.05 0)
-      (effects (font (size 1.27 1.27)) hide)
-    )
-    (property "Function" "SPI Power DDC/i2c ROM" (at 106.68 142.24 0)
+  (symbol (lib_id "Connector_Generic:Conn_01x02") (at 104.14 144.78 0) (unit 1)
+    (in_bom yes) (on_board yes) (dnp no)
+    (property "Reference" "JP1" (at 106.68 146.05 0)
+      (effects (font (size 1.27 1.27)) (justify left))
+    )
+    (property "Value" "DDC 5V" (at 106.68 147.955 0)
+      (effects (font (size 1.27 1.27)) (justify left))
+    )
+    (property "Footprint" "Connector_PinHeader_2.54mm:PinHeader_1x02_P2.54mm_Vertical" (at 104.14 144.78 0)
+      (effects (font (size 1.27 1.27)) hide)
+    )
+    (property "Datasheet" "~" (at 104.14 144.78 0)
+      (effects (font (size 1.27 1.27)) hide)
+    )
+    (property "Function" "SPI Power DDC/i2c ROM" (at 114.3 137.16 0)
       (effects (font (size 1.27 1.27)))
     )
@@
     )
   )
-  (symbol (lib_id "power:VCC") (at 88.9 143.51 0) (unit 1)
+  (symbol (lib_id "power:VCC") (at 97.79 142.24 0) (unit 1)
     (in_bom yes) (on_board yes) (dnp no) (fields_autoplaced)
-    (property "Reference" "#PWR019" (at 88.9 147.32 0)
-      (effects (font (size 1.27 1.27)) hide)
-    )
-    (property "Value" "VCC" (at 88.9 139.7 0)
+    (property "Reference" "#PWR019" (at 97.79 146.05 0)
+      (effects (font (size 1.27 1.27)) hide)
+    )
+    (property "Value" "VCC" (at 97.79 138.43 0)
       (effects (font (size 1.27 1.27)))
     )
-    (property "Footprint" "" (at 88.9 143.51 0)
-      (effects (font (size 1.27 1.27)) hide)
-    )
-    (property "Datasheet" "" (at 88.9 143.51 0)
+    (property "Footprint" "" (at 97.79 142.24 0)
+      (effects (font (size 1.27 1.27)) hide)
+    )
+    (property "Datasheet" "" (at 97.79 142.24 0)
       (effects (font (size 1.27 1.27)) hide)
     )
@@
         )
       )
+    )
+  )
+  (symbol (lib_id "Device:R") (at 95.25 147.32 90) (mirror x) (unit 1)
+    (in_bom yes) (on_board yes) (dnp no)
+    (property "Reference" "R48" (at 96.52 144.78 90)
+      (effects (font (size 1.27 1.27)) (justify left))
+    )
+    (property "Value" "33R" (at 96.52 149.86 90)
+      (effects (font (size 1.27 1.27)) (justify left))
+    )
+    (property "Footprint" "Resistor_SMD:R_0805_2012Metric_Pad1.20x1.40mm_HandSolder" (at 95.25 145.542 90)
+      (effects (font (size 1.27 1.27)) hide)
+    )
+    (property "Datasheet" "~" (at 95.25 147.32 0)
+      (effects (font (size 1.27 1.27)) hide)
+    )
+    (pin "1")
+    (pin "2")
+    (instances
+      (project "virge-vlb"
+        (path "/e8216711-86b5-4276-82f4-4c7ed22b9a9c"
+          (reference "R48") (unit 1)
+        )
+      )
