File: kicad/address.kicad_sch (KiCad schematic)
At the start: 11 parts, among them J1 VLB_slot, U1 86C325, U8 7404, U9 7408

Commit message: changed QFP and ROM footprint
Parts:
- U1: footprint Package_QFP:PQFP-208_28x28mm_P0.5mm -> VLB:QFP-208
Changed lines of the file:
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@@
       (effects (font (size 1.524 1.524)))
     )
-    (property "Footprint" "Package_QFP:PQFP-208_28x28mm_P0.5mm" (at 20.32 115.57 0)
+    (property "Footprint" "VLB:QFP-208" (at 20.32 115.57 0)
       (effects (font (size 1.524 1.524)) (justify right) hide)
     )
@@
       (effects (font (size 1.524 1.524)) (justify left))
     )
-    (property "Footprint" "Package_QFP:PQFP-208_28x28mm_P0.5mm" (at 107.95 142.24 0)
+    (property "Footprint" "VLB:QFP-208" (at 107.95 142.24 0)
       (effects (font (size 1.524 1.524)) (justify right) hide)
     )
@@
       (effects (font (size 1.524 1.524)))
     )
-    (property "Footprint" "Package_QFP:PQFP-208_28x28mm_P0.5mm" (at 21.59 165.1 0)
+    (property "Footprint" "VLB:QFP-208" (at 21.59 165.1 0)
       (effects (font (size 1.524 1.524)) (justify right) hide)
     )
