File: kicad/address.kicad_sch (KiCad schematic)
At the start: 12 parts, among them J1 VLB_slot, U10 86C765, U8 7404, U9 7408

Commit message: updated to kicad 9
Parts:
- renumbered C14 to C11, C19 to C15, C20 to C18, JP3 to JP4, R5 to R4, R5 to R47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
