File: kicad/data.kicad_sch (KiCad schematic)
At the start: 39 parts, among them U7 86C325

Commit message: changed QFP and ROM footprint
Parts:
- R5: value 33R -> 2 x 33R
- U7: footprint Package_QFP:PQFP-208_28x28mm_P0.5mm -> VLB:QFP-208
Changed lines of the file:
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@@
       (effects (font (size 1.27 1.27)) (justify left))
     )
-    (property "Value" "33R" (at 40.64 180.34 90)
+    (property "Value" "2 x 33R" (at 40.64 180.34 90)
       (effects (font (size 1.27 1.27)) (justify left) hide)
     )
@@
       (effects (font (size 1.524 1.524)) (justify left))
     )
-    (property "Footprint" "Package_QFP:PQFP-208_28x28mm_P0.5mm" (at 19.05 158.75 0)
+    (property "Footprint" "VLB:QFP-208" (at 19.05 158.75 0)
       (effects (font (size 1.524 1.524)) (justify right) hide)
     )
@@
       (effects (font (size 1.524 1.524)))
     )
-    (property "Footprint" "Package_QFP:PQFP-208_28x28mm_P0.5mm" (at 5.08 78.74 0)
+    (property "Footprint" "VLB:QFP-208" (at 5.08 78.74 0)
       (effects (font (size 1.524 1.524)) (justify right) hide)
     )
@@
       (effects (font (size 1.524 1.524)) (justify left))
     )
-    (property "Footprint" "Package_QFP:PQFP-208_28x28mm_P0.5mm" (at 83.82 157.48 0)
+    (property "Footprint" "VLB:QFP-208" (at 83.82 157.48 0)
       (effects (font (size 1.524 1.524)) (justify right) hide)
     )
