File: kicad/_autosave-address.kicad_sch (KiCad schematic)
At the start: 11 parts, among them J1 VLB_slot, U1 86C325, U8 7404, U9 7408

Commit message: some polishing
Changed lines of the file:
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@@
     (fill (type none))
-  )
-  (text_box "C15, reduce to 1 or 10nF depending on tested board parameters. (Reset stability)"
-    (at 127 170.18 0) (size 22.86 13.97)
-    (stroke (width 0) (type default))
-    (fill (type none))
-    (effects (font (size 1.27 1.27)) (justify left top))
   )
   (text "SAUP address decoding" (at 19.05 19.05 0)
