File: kicad/_autosave-data.kicad_sch (KiCad schematic)
At the start: 39 parts, among them U7 86C325

Commit message: some polishing
Other:
- note added: "Register configurations: (see pages 46-47 in the 64V+/ViRGE doc)"
- note removed: "Register configurations: (see pages 46-47 in the ViRGE doc)"
Changed lines of the file:
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@@
     (fill (type none))
   )
-  (text_box "R6-R16 Series Termination 33 Ohm\nAdjust based on PCB final prod characteristics"
+  (text_box "R10-R21 Series Termination 33 Ohm\nAdjust based on PCB final prod characteristics"
     (at 69.85 149.86 0) (size 27.94 11.2522)
     (stroke (width 0) (type default))
@@
     (effects (font (size 1.27 1.27)) (justify left bottom))
   )
-  (text "Register configurations:\n(see pages 46-47 in the ViRGE doc)"
+  (text "Register configurations:\n(see pages 46-47 in the 64V+/ViRGE doc)"
     (at 154.94 19.05 0)
     (effects (font (size 1.27 1.27)) (justify left bottom))
