File: kicad/virge-vlb.kicad_sch (KiCad schematic)
At the start: 39 parts, among them CN1 VGA, U1 86C325, Y1 14.318MHz

Commit message: some final tweaks
Parts:
- removed C20: 10uF, Capacitor_SMD:C_1206_3216Metric_Pad1.33x1.80mm_HandSolder, symbol Device:C_Polarized
- removed R11, R9: 33R, Resistor_SMD:R_0805_2012Metric_Pad1.20x1.40mm_HandSolder, symbol Device:R
- removed R22: 10K, Resistor_SMD:R_0805_2012Metric_Pad1.20x1.40mm_HandSolder, symbol Device:R
- removed R45: 4.7K, Resistor_SMD:R_0805_2012Metric_Pad1.20x1.40mm_HandSolder, symbol Device:R
- added C10, C9: 10pF, Capacitor_SMD:C_0805_2012Metric_Pad1.18x1.45mm_HandSolder, symbol Device:C
- added C30: 10uF, Capacitor_SMD:C_1206_3216Metric_Pad1.33x1.80mm_HandSolder, symbol Device:C_Polarized
- added R20, R21: 33R, Resistor_SMD:R_0805_2012Metric_Pad1.20x1.40mm_HandSolder, symbol Device:R
- added R43: 10K, Resistor_SMD:R_0805_2012Metric_Pad1.20x1.40mm_HandSolder, symbol Device:R
- R44: value 4.7K -> 10K
- renumbered C3 to C1, C4 to C2, C5 to C3, C6 to C4, C7 to C5, C8 to C6, C1 to C7, C2 to C8, FB3 to FB2, FB2 to FB3, R3 to R1, R4 to R2, R42 to R22, R5 to R3, R43 to R42, R46 to R45, R1 to R7, R2 to R8
Connections:
- net DDC_SDA_VGA is gone; now on an unnamed net: CN1.12
- net DDC_SCL: now also R21.1; no longer R44.1
- net DDC_SDA: now also R20.1
- net GND: now also C10.1, C30.2, C9.1
- net VCC: now also R44.1, C30.1, R43.1
- net at JP1.2 (Pin_2): now also CN1.9
- net at U1.156 (XIN), Y1.2: now also C9.2
- net at U1.157 (XOUT), Y1.1: now also C10.2
- net DDC_SCL_VGA: no longer names the net of R44.2
- net DDC_SCL_VGA: now also R20.2; no longer CN1.15
- new net: CN1.15, R21.2, R43.2
Other:
- note removed: "DDC I2C Bus"
- moved on the sheet: C21, C22, C23, C24, C25, C26, C27, C28, C29, C4, C5, C6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

Commit message: added pull up, new BOM
Parts:
- added R43: 10K, Resistor_SMD:R_0805_2012Metric_Pad1.20x1.40mm_HandSolder, symbol Device:R
- renumbered R42 to R22, R22 to R42, R43 to R45, R45 to R46
Connections:
- net VCC: now also R43.2
- net at R42.1, U1.204 (~{CREQ}/CRDY/EVCLK): no longer U1.203 (~{VREQ}/VRDY/EVIDEO)
- new net: R43.1, U1.203 (~{VREQ}/VRDY/EVIDEO)
Other:
- moved on the sheet: R42
Changed lines of the file:
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@@
   (junction (at 40.64 146.05) (diameter 0) (color 0 0 0 0)
   )
-  (junction (at 173.99 69.85) (diameter 0) (color 0 0 0 0)
-  )
   (junction (at 111.76 151.13) (diameter 0) (color 0 0 0 0)
   )
@@
   )
   (junction (at 40.64 34.29) (diameter 0) (color 0 0 0 0)
+  )
+  (junction (at 151.13 68.58) (diameter 0) (color 0 0 0 0)
   )
   (junction (at 36.83 151.13) (diameter 0) (color 0 0 0 0)
@@
     (stroke (width 0) (type default))
   )
+  (wire (pts (xy 162.56 67.31) (xy 162.56 68.58))
+    (stroke (width 0) (type default))
+  )
   (wire (pts (xy 78.74 140.97) (xy 83.82 140.97))
     (stroke (width 0) (type default))
@@
     (stroke (width 0) (type default))
   )
-  (wire (pts (xy 173.99 67.31) (xy 173.99 69.85))
+  (wire (pts (xy 163.83 73.66) (xy 163.83 69.85))
     (stroke (width 0) (type default))
   )
@@
     (stroke (width 0) (type default))
   )
+  (wire (pts (xy 163.83 69.85) (xy 173.99 69.85))
+    (stroke (width 0) (type default))
+  )
   (wire (pts (xy 139.7 177.8) (xy 144.78 177.8))
     (stroke (width 0) (type default))
@@
     (stroke (width 0) (type default))
   )
-  (wire (pts (xy 151.13 69.85) (xy 151.13 66.04))
+  (wire (pts (xy 151.13 73.66) (xy 151.13 68.58))
     (stroke (width 0) (type default))
   )
@@
     (stroke (width 0) (type default))
   )
+  (wire (pts (xy 173.99 67.31) (xy 162.56 67.31))
+    (stroke (width 0) (type default))
+  )
   (wire (pts (xy 127 189.23) (xy 127 186.69))
     (stroke (width 0) (type default))
@@
     (stroke (width 0) (type default))
   )
+  (wire (pts (xy 151.13 68.58) (xy 151.13 66.04))
+    (stroke (width 0) (type default))
+  )
   (wire (pts (xy 124.46 151.13) (xy 153.67 151.13))
     (stroke (width 0) (type default))
@@
     (stroke (width 0) (type default))
   )
-  (wire (pts (xy 154.94 69.85) (xy 151.13 69.85))
+  (wire (pts (xy 154.94 73.66) (xy 151.13 73.66))
     (stroke (width 0) (type default))
   )
@@
     (stroke (width 0) (type default))
   )
-  (wire (pts (xy 162.56 69.85) (xy 173.99 69.85))
+  (wire (pts (xy 162.56 73.66) (xy 163.83 73.66))
+    (stroke (width 0) (type default))
+  )
+  (wire (pts (xy 151.13 68.58) (xy 154.94 68.58))
     (stroke (width 0) (type default))
   )
@@
   (symbol (lib_id "Device:R") (at 55.88 137.16 0) (mirror y) (unit 1)
     (in_bom yes) (on_board yes) (dnp no)
-    (property "Reference" "R43" (at 60.96 134.62 0)
+    (property "Reference" "R45" (at 60.96 134.62 0)
       (effects (font (size 1.27 1.27)) (justify left))
     )
@@
       (project "virge-vlb"
         (path "/e8216711-86b5-4276-82f4-4c7ed22b9a9c"
-          (reference "R43") (unit 1)
+          (reference "R45") (unit 1)
         )
       )
@@
     )
   )
-  (symbol (lib_id "Device:R") (at 158.75 69.85 270) (unit 1)
-    (in_bom yes) (on_board yes) (dnp no)
-    (property "Reference" "R22" (at 157.48 67.31 90)
-      (effects (font (size 1.27 1.27)) (justify left))
-    )
-    (property "Value" "10K" (at 157.48 72.39 90)
-      (effects (font (size 1.27 1.27)) (justify left))
-    )
-    (property "Footprint" "Resistor_SMD:R_0805_2012Metric_Pad1.20x1.40mm_HandSolder" (at 158.75 68.072 90)
-      (effects (font (size 1.27 1.27)) hide)
-    )
-    (property "Datasheet" "~" (at 158.75 69.85 0)
-      (effects (font (size 1.27 1.27)) hide)
-    )
-    (pin "1")
-    (pin "2")
-    (instances
-      (project "virge-vlb"
-        (path "/e8216711-86b5-4276-82f4-4c7ed22b9a9c"
-          (reference "R22") (unit 1)
+  (symbol (lib_id "Device:R") (at 158.75 73.66 270) (unit 1)
+    (in_bom yes) (on_board yes) (dnp no)
+    (property "Reference" "R42" (at 157.48 71.12 90)
+      (effects (font (size 1.27 1.27)) (justify left))
+    )
+    (property "Value" "10K" (at 157.48 73.66 90)
+      (effects (font (size 1.27 1.27)) (justify left))
+    )
+    (property "Footprint" "Resistor_SMD:R_0805_2012Metric_Pad1.20x1.40mm_HandSolder" (at 158.75 71.882 90)
+      (effects (font (size 1.27 1.27)) hide)
+    )
+    (property "Datasheet" "~" (at 158.75 73.66 0)
+      (effects (font (size 1.27 1.27)) hide)
+    )
+    (pin "1")
+    (pin "2")
+    (instances
+      (project "virge-vlb"
+        (path "/e8216711-86b5-4276-82f4-4c7ed22b9a9c"
+          (reference "R42") (unit 1)
         )
         (path "/e8216711-86b5-4276-82f4-4c7ed22b9a9c/73bb2a59-bfac-4efc-8051-53849b0f9066"
@@
         (path "/e8216711-86b5-4276-82f4-4c7ed22b9a9c"
           (reference "C26") (unit 1)
+        )
+      )
+    )
+  )
+  (symbol (lib_id "Device:R") (at 158.75 68.58 270) (unit 1)
+    (in_bom yes) (on_board yes) (dnp no)
+    (property "Reference" "R43" (at 157.48 66.04 90)
+      (effects (font (size 1.27 1.27)) (justify left))
+    )
+    (property "Value" "10K" (at 157.48 68.58 90)
+      (effects (font (size 1.27 1.27)) (justify left))
+    )
+    (property "Footprint" "Resistor_SMD:R_0805_2012Metric_Pad1.20x1.40mm_HandSolder" (at 158.75 66.802 90)
+      (effects (font (size 1.27 1.27)) hide)
+    )
+    (property "Datasheet" "~" (at 158.75 68.58 0)
+      (effects (font (size 1.27 1.27)) hide)
+    )
+    (pin "1")
+    (pin "2")
+    (instances
+      (project "virge-vlb"
+        (path "/e8216711-86b5-4276-82f4-4c7ed22b9a9c"
+          (reference "R43") (unit 1)
+        )
+        (path "/e8216711-86b5-4276-82f4-4c7ed22b9a9c/73bb2a59-bfac-4efc-8051-53849b0f9066"
+          (reference "R16") (unit 1)
         )
       )
@@
   (symbol (lib_id "Device:R") (at 212.09 77.47 270) (unit 1)
     (in_bom yes) (on_board yes) (dnp no)
-    (property "Reference" "R45" (at 210.82 74.93 90)
+    (property "Reference" "R46" (at 210.82 74.93 90)
       (effects (font (size 1.27 1.27)) (justify left))
     )
@@
       (project "virge-vlb"
         (path "/e8216711-86b5-4276-82f4-4c7ed22b9a9c"
-          (reference "R45") (unit 1)
+          (reference "R46") (unit 1)
         )
         (path "/e8216711-86b5-4276-82f4-4c7ed22b9a9c/73bb2a59-bfac-4efc-8051-53849b0f9066"
@@
   (symbol (lib_id "Device:R") (at 158.75 57.15 270) (unit 1)
     (in_bom yes) (on_board yes) (dnp no)
-    (property "Reference" "R42" (at 157.48 54.61 90)
+    (property "Reference" "R22" (at 157.48 54.61 90)
       (effects (font (size 1.27 1.27)) (justify left))
     )
@@
       (project "virge-vlb"
         (path "/e8216711-86b5-4276-82f4-4c7ed22b9a9c"
-          (reference "R42") (unit 1)
+          (reference "R22") (unit 1)
         )
         (path "/e8216711-86b5-4276-82f4-4c7ed22b9a9c/73bb2a59-bfac-4efc-8051-53849b0f9066"

Commit message: many fixes for rev 1C
Other:
- moved on the sheet: R42
