File: kicad/busctrl.kicad_sch (KiCad schematic)
At the start: 7 parts, among them J1 VLB_slot, U1 74LS245, U2 27C020

Commit message: fixed VGA footprint
Parts:
- J1: footprint (none) -> VLB:BUS_VLB_Board
Changed lines of the file:
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@@
       (effects (font (size 1.27 1.27)))
     )
-    (property "Footprint" "" (at 139.7 80.01 0)
+    (property "Footprint" "VLB:BUS_VLB_Board" (at 139.7 80.01 0)
       (effects (font (size 1.27 1.27)) hide)
     )

Commit message: final fixes
Connections:
- net GND: now also U1.1 (A->B)
Changed lines of the file:
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@@
+    (stroke (width 0) (type default))
+  )
+  (wire (pts (xy 45.72 92.71) (xy 57.15 92.71))
     (stroke (width 0) (type default))
   )
@@
         )
       )
+    )
+  )
+  (symbol (lib_id "power:GND") (at 45.72 92.71 0) (unit 1)
+    (in_bom yes) (on_board yes) (dnp no) (fields_autoplaced)
+    (property "Reference" "#PWR062" (at 45.72 99.06 0)
+      (effects (font (size 1.27 1.27)) hide)
+    )
+    (property "Value" "GND" (at 45.72 97.79 0)
+      (effects (font (size 1.27 1.27)))
+    )
+    (property "Footprint" "" (at 45.72 92.71 0)
+      (effects (font (size 1.27 1.27)) hide)
+    )
+    (property "Datasheet" "" (at 45.72 92.71 0)
+      (effects (font (size 1.27 1.27)) hide)
+    )
+    (pin "1")
+    (instances
+      (project "virge-vlb"
+        (path "/e8216711-86b5-4276-82f4-4c7ed22b9a9c/485e825d-a3d2-4e3d-9ea7-d005dd511bf5"
+          (reference "#PWR062") (unit 1)
+        )
+        (path "/e8216711-86b5-4276-82f4-4c7ed22b9a9c/9321f466-5ac6-411a-b039-07fb7f0cdeaa"
+          (reference "#PWR024") (unit 1)
+        )
+      )

Commit message: fix for LS245 bus conflict
Connections:
- net GND: no longer U1.1 (A->B)
- net SMEMR: now also U1.1 (A->B)
Changed lines of the file:
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@@
-    (stroke (width 0) (type default))
-  )
-  (wire (pts (xy 45.72 92.71) (xy 57.15 92.71))
     (stroke (width 0) (type default))
   )
@@
     (stroke (width 0) (type default))
   )
+  (wire (pts (xy 49.53 92.71) (xy 57.15 92.71))
+    (stroke (width 0) (type default))
+  )
   (wire (pts (xy 129.54 72.39) (xy 137.16 72.39))
     (stroke (width 0) (type default))
@@
   )
   (label "ISA_D6" (at 49.53 85.09 0) (fields_autoplaced)
+    (effects (font (size 1.27 1.27)) (justify left bottom))
+  )
+  (label "SMEMR" (at 49.53 92.71 0) (fields_autoplaced)
     (effects (font (size 1.27 1.27)) (justify left bottom))
   )
@@
         )
       )
-    )
-  )
-  (symbol (lib_id "power:GND") (at 45.72 92.71 0) (unit 1)
-    (in_bom yes) (on_board yes) (dnp no) (fields_autoplaced)
-    (property "Reference" "#PWR062" (at 45.72 99.06 0)
-      (effects (font (size 1.27 1.27)) hide)
-    )
-    (property "Value" "GND" (at 45.72 97.79 0)
-      (effects (font (size 1.27 1.27)))
-    )
-    (property "Footprint" "" (at 45.72 92.71 0)
-      (effects (font (size 1.27 1.27)) hide)
-    )
-    (property "Datasheet" "" (at 45.72 92.71 0)
-      (effects (font (size 1.27 1.27)) hide)
-    )
-    (pin "1")
-    (instances
-      (project "virge-vlb"
-        (path "/e8216711-86b5-4276-82f4-4c7ed22b9a9c/485e825d-a3d2-4e3d-9ea7-d005dd511bf5"
-          (reference "#PWR062") (unit 1)
-        )
-        (path "/e8216711-86b5-4276-82f4-4c7ed22b9a9c/9321f466-5ac6-411a-b039-07fb7f0cdeaa"
-          (reference "#PWR024") (unit 1)
-        )
-      )

Commit message: updated to kicad 9
Parts:
- renumbered C14 to C17
